Commit message: forgot to commit

File: src/iiwa_stack/iiwa_description/urdf/backup/iiwa7.xacro (robot description, xacro)
@@ -11,6 +11,6 @@
   <xacro:property name="safety_controller_k_vel" value="20000" />
   <xacro:property name="joint_damping" value="0.5" />
-  <xacro:property name="max_effort" value="300000"/>
-  <xacro:property name="max_velocity" value="1000"/>
+  <xacro:property name="max_effort" value="3000"/>
+  <xacro:property name="max_velocity" value="50"/>
   <xacro:macro name="iiwa7" params="parent hardware_interface robot_name *origin">
     <!--joint between {parent} and link_0-->

File: src/iiwa_stack/iiwa_tool_description/urdf/iiwa_tool.urdf.xacro (robot description, xacro)
@@ -39,7 +39,7 @@
   </xacro:iiwa7>
   <!-- Tool properties -->
-  <property name="tool_mass" value="0.200" />
+  <property name="tool_mass" value="0.070" />
   <property name="tool_joint_offset" value="0.00 0.00 0.00" />
-  <property name="tool_link_offset" value="0.00 0.00 0.1275" />
+  <property name="tool_link_offset" value="0.00 0.00 0.135" />
   <!--  Here we define a dummy joint between the tip of the iiwa7 and the base of the tool.
   There is no offset between the two, that means the tool is attached at the robot flange. -->
