Commit message: added autonomous ball returning

File: src/iiwa_stack/iiwa_tool_description/urdf/iiwa_tool.urdf.xacro (robot description, xacro)
@@ -2,58 +2,79 @@
 <!-- Here we define the robot, we named it "iiwa7_tool" -->
 <robot xmlns:xacro="http://www.ros.org/wiki/xacro" name="iiwa7_tool">
-  <!-- Import Rviz colors -->
-  <xacro:include filename="$(find iiwa_description)/urdf/materials.xacro" />
-  <!--Import the iiwa7 macro -->
-  <xacro:include filename="$(find iiwa_description)/urdf/iiwa7.xacro"/>
-  <!--  Arguments for the iiwa7 macro  -->
-  <xacro:arg name="hardware_interface" default="PositionJointInterface"/>
-  <xacro:arg name="robot_name" default="iiwa"/>
-  <!--  Define the origin of your 3D space
+    <!-- Import Rviz colors -->
+    <xacro:include filename="$(find iiwa_description)/urdf/materials.xacro" />
+    <!--Import the iiwa7 macro -->
+    <xacro:include filename="$(find iiwa_description)/urdf/iiwa7.xacro"/>
+    <!--  Arguments for the iiwa7 macro  -->
+    <xacro:arg name="hardware_interface" default="PositionJointInterface"/>
+    <xacro:arg name="robot_name" default="iiwa"/>
+    <!--  Define the origin of your 3D space
   Here we define a box lying at 0,0,0 with some dimensions, in reality our robot is place on top of a metal cart with those dimensions.
   This will include the cart in the scene and avoid the robot to hit it when using MoveIt!
   If you don't want to have that you can define a basic world link (see commented lines)
   -->
-  <link name="world"/>
-  <gazebo reference="world">
-    <static>true</static>
-  </gazebo>
-  <!-- Here we insert an iiwa7 robot in the scene, it's origin is just on top of the box previously defined. You can use 0,0,0 if you don't have that. -->
-  <xacro:iiwa7 hardware_interface="$(arg hardware_interface)" robot_name="$(arg robot_name)" parent="world">
-    <origin xyz="0 0 0" rpy="0 0 0"/>
-  </xacro:iiwa7>
-  <!-- Tool properties -->
-  <property name="tool_mass" value="0.070" />
-  <property name="tool_joint_offset" value="0.00 0.00 0.00" />
-  <property name="tool_link_offset" value="0.00 0.00 0.135" />
-  <!--  Here we define a dummy joint between the tip of the iiwa7 and the base of the tool.
+    <link name="world"/>
+    <gazebo reference="world">
+        <static>true</static>
+    </gazebo>
+    <!-- Here we insert an iiwa7 robot in the scene, it's origin is just on top of the box previously defined. You can use 0,0,0 if you don't have that. -->
+    <xacro:iiwa7 hardware_interface="$(arg hardware_interface)" robot_name="$(arg robot_name)" parent="world">
+        <origin xyz="0 0 0" rpy="0 0 0"/>
+    </xacro:iiwa7>
+    <!-- Tool properties -->
+    <property name="tool_mass" value="0.070" />
+    <property name="tool_joint_offset" value="0.00 0.00 0.00" />
+    <property name="tool_link_offset" value="0.00 0.00 0.135" />
+    <!--  Here we define a dummy joint between the tip of the iiwa7 and the base of the tool.
   There is no offset between the two, that means the tool is attached at the robot flange. -->
-  <joint name="tool_joint" type="fixed">
-    <parent link="iiwa_link_ee" />
-    <child link = "tool_link" />
-    <origin xyz="${tool_joint_offset}" rpy="0 0 -${PI/2.0}" />
-  </joint>
-  <!-- Here we define the geometry of the tool. We designed the tool ourselves, so we have a mesh file that represents it.
+    <joint name="tool_joint" type="fixed">
+        <parent link="iiwa_link_ee" />
+        <child link = "tool_link" />
+        <origin xyz="${tool_joint_offset}" rpy="0 0 -${PI/2.0}" />
+    </joint>
+    <!-- Here we define the geometry of the tool. We designed the tool ourselves, so we have a mesh file that represents it.
   Else, one can define it using a geometric representation that approximate it, like a cylinder (see commented lines) -->
-  <link name="tool_link">
-    <visual>
-      <origin xyz="0 0 0" rpy="0 0 0"/>
-      <geometry>
-    	<mesh filename="package://iiwa_tool_description/meshes/visual/racket.dae"/>
-      </geometry>
-    </visual>
-    <collision name="racket_collision">
-      <origin xyz="0 0 0" rpy="0 0 0"/>
-      <geometry>
-        <mesh filename="package://iiwa_tool_description/meshes/visual/racket.dae"/>
-      </geometry>
-    </collision>
-  </link>
-  <!--  Here we define another dummy joint. It is placed at the end of the tool, so we can then attach a frame at its TCP for control -->
-  <joint name="tool_tip_joint" type="fixed">
-    <parent link="tool_link" />
-    <child link = "tool_link_ee" />
-    <origin xyz="${tool_link_offset}" rpy="0 0 0" />
-  </joint>
-  <!--  The TCP frame is here defined -->
-  <link name="tool_link_ee"/>
+    <link name="tool_link">
+        <visual>
+            <origin xyz="0 0 0" rpy="0 0 0"/>
+            <geometry>
+                <mesh filename="package://iiwa_tool_description/meshes/visual/racket.dae"/>
+            </geometry>
+        </visual>
+        <collision name="racket_collision">
+            <origin xyz="0 0 0" rpy="0 0 0"/>
+            <geometry>
+                <mesh filename="package://iiwa_tool_description/meshes/visual/racket.dae"/>
+            </geometry>
+        </collision>
+    </link>
+    <gazebo reference="iiwa_link_7">
+        <collision name="racket_collision">
+            <surface>
+                <bounce>
+                    <restitution_coefficient>0.75</restitution_coefficient>
+                    <threshold>0</threshold>
+                </bounce>
+                <friction>
+                    <ode>
+                        <mu>0.01</mu>
+                        <mu2>0.01</mu2>
+                    </ode>
+                </friction>
+                <contact>
+                    <ode>
+                        <max_vel>1000</max_vel>
+                    </ode>
+                </contact>
+            </surface>
+        </collision>
+    </gazebo>
+    <!--  Here we define another dummy joint. It is placed at the end of the tool, so we can then attach a frame at its TCP for control -->
+    <joint name="tool_tip_joint" type="fixed">
+        <parent link="tool_link" />
+        <child link = "tool_link_ee" />
+        <origin xyz="${tool_link_offset}" rpy="0 0 0" />
+    </joint>
+    <!--  The TCP frame is here defined -->
+    <link name="tool_link_ee"/>
 </robot>
